Commit message: Updated masses in some of our models

File: src/brom_drake/robots/models/beaker/beaker.urdf (robot description, URDF)
Before this commit: robot beaker, 1 links, 0 joints
Links:
- link beaker_base_link: mass None -> 2.5

File: src/brom_drake/robots/models/test_tube_holder/test_tube_holder.urdf (robot description, URDF)
Before this commit: robot test-tube-holder, 1 links, 0 joints
Links:
- link test_tube_holder_base_link: mass None -> 1.0
