Commit message: wip: Almost debugged grasping production

File: src/brom_drake/robots/models/erlenmeyer_flask/500ml.urdf (robot description, URDF)
Before this commit: robot erlenmeyer_flask_500ml, 1 links, 0 joints
Links:
- link flask_base_link: mass 5.0 -> 0.5445761924742986

Commit message: changed the suffix of the stl file for the 500ml urdf

File: src/brom_drake/robots/models/erlenmeyer_flask/500ml.urdf (robot description, URDF)
Before this commit: robot erlenmeyer_flask_500ml, 1 links, 0 joints
Links:
- link flask_base_link: geometry collision mesh filename=500ml.stl scale=0.001 0.001 0.001; visual mesh filename=500ml.stl scale=0.001 0.001 0.001

Commit message: Reverted reference in the urdf to use capitals again?

File: src/brom_drake/robots/models/erlenmeyer_flask/500ml.urdf (robot description, URDF)
Before this commit: robot erlenmeyer_flask_500ml, 1 links, 0 joints
Links:
- link flask_base_link: geometry collision mesh filename=500ml.STL scale=0.001 0.001 0.001; visual mesh filename=500ml.STL scale=0.001 0.001 0.001
