Commit message: small path updates to URDF

File: tests/file_manipulation/urdf/DrakeReadyURDFConverter/resources/test5_absolute.urdf (robot description, URDF)
Before this commit: robot test-robot, 1 links, 0 joints
Links:
- link base_link_inertia: geometry collision mesh filename=file:///workspaces/brom_drake-py/tests/file_manipulation/ur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; visual mesh filename=file:///workspaces/brom_drake-py/tests/file_manipulation/ur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
